Commit message: spot naprawa

File: install/rover_description/share/rover_description/urdf/Rover.xacro (robot description, xacro)
@@ -1 +1,1397 @@
-/home/pawla/ros2_ws/src/rover_description/rover_description/urdf/Rover.xacro
+<?xml version="1.0" ?>
+<robot name="Rover" xmlns:xacro="http://www.ros.org/wiki/xacro">
+  <xacro:arg name="sim" default="true"/>
+  <xacro:arg name="controllers_file"
+             default="$(find rover_description)/config/controllers.yaml"/>
+<xacro:include filename="$(find rover_description)/urdf/materials.xacro" />
+<xacro:include filename="$(find rover_description)/urdf/Rover.trans" />
+<xacro:include filename="$(find rover_description)/urdf/Rover.gazebo" />
+<link name="base_footprint"/>
+<joint name="base_footprint_joint" type="fixed">
+  <parent link="base_footprint"/>
+  <child link="base_link"/>
+  <origin xyz="0 0 0.27" rpy="0 0 -1.5708"/>
+</joint>
+<link name="base_link">
+  <inertial>
+    <origin xyz="-3.3708776575841558e-15 0.00363761455711936 0.007362716562946554" rpy="0 0 0"/>
+    <mass value="0.3844784894849203"/>
+    <inertia ixx="0.002117" iyy="0.001" izz="0.002775" ixy="0.0" iyz="-0.0" ixz="-0.0"/>
+  </inertial>
+  <visual>
+    <origin xyz="0 0 0" rpy="0 0 0"/>
+    <geometry>
+      <mesh filename="package://rover_description/meshes/base_link.stl" scale="0.001 0.001 0.001"/>
+    </geometry>
+    <material name="silver"/>
+  </visual>
+  <collision>
+    <origin xyz="0 0.05 0" rpy="0 0 0"/>
+    <geometry>
+      <box size="0.375 0.52 0.25"/>
+    </geometry>
+  </collision>
+</link>
+<link name="pret_handler_v3proba_v1_1">
+  <inertial>
+    <origin xyz="-0.01900000000000006 -4.143233196599039e-07 -0.005389574608387276" rpy="0 0 0"/>
+    <mass value="0.11371542799884354"/>
+    <inertia ixx="0.000221" iyy="0.001" izz="0.001" ixy="-0.0" iyz="0.0" ixz="0.0"/>
+  </inertial>
+  <visual>
+    <origin xyz="0.094 0.05475 -0.033612" rpy="0 0 0"/>
+    <geometry>
+      <mesh filename="package://rover_description/meshes/pret_handler_v3proba_v1_1.stl" scale="0.001 0.001 0.001"/>
+    </geometry>
+    <material name="silver"/>
+  </visual>
+  <!-- <collision>
+    <origin xyz="0.094 0.05475 -0.033612" rpy="0 0 0"/>
+    <geometry>
+      <box size="0.236 0.035 0.0585"/>
+    </geometry>
+  </collision> -->
+</link>
+<link name="pret_handler_v3proba_v1__1__1">
+  <inertial>
+    <origin xyz="0.01899999999999999 -4.143232613593173e-07 -0.005389574608387286" rpy="0 0 0"/>
+    <mass value="0.11371542799884354"/>
+    <inertia ixx="0.000221" iyy="0.001" izz="0.001" ixy="-0.0" iyz="-0.0" ixz="0.0"/>
+  </inertial>
+  <visual>
+    <origin xyz="-0.094 0.05475 -0.033612" rpy="0 0 0"/>
+    <geometry>
+      <mesh filename="package://rover_description/meshes/pret_handler_v3proba_v1__1__1.stl" scale="0.001 0.001 0.001"/>
+    </geometry>
+    <material name="silver"/>
+  </visual>
+  <!-- <collision>
+    <origin xyz="-0.094 0.05475 -0.033612" rpy="0 0 0"/>
+    <geometry>
+      <box size="0.236 0.035 0.0585"/>
+    </geometry>
+  </collision> -->
+</link>
+<link name="handler_backv2proba_v1_1">
+  <inertial>
+    <origin xyz="-7.126086628479645e-05 0.04736205845248642 -0.005801507049937215" rpy="0 0 0"/>
+    <mass value="0.20973987708628855"/>
+    <inertia ixx="0.001" iyy="0.000708" izz="0.000907" ixy="0.0" iyz="2e-06" ixz="1e-05"/>
+  </inertial>
+  <visual>
+    <origin xyz="0.0 -0.155316 -0.033612" rpy="0 0 0"/>
+    <geometry>
+      <mesh filename="package://rover_description/meshes/handler_backv2proba_v1_1.stl" scale="0.001 0.001 0.001"/>
+    </geometry>
+    <material name="silver"/>
+  </visual>
+  <!-- <collision>
+    <origin xyz="0.0 -0.155316 -0.033612" rpy="0 0 0"/>
+    <geometry>
+      <box size="0.31 0.104 0.035"/>
+    </geometry>
+  </collision> -->
+</link>
+<link name="basketback_v1_1">
+  <inertial>
+    <origin xyz="-0.026262275115844294 -4.143231134845493e-07 -0.0014781940855226675" rpy="0 0 0"/>
+    <mass value="0.05211230478294979"/>
+    <inertia ixx="0.001" iyy="0.001" izz="0.001" ixy="0.0" iyz="0.0" ixz="0.0"/>
+  </inertial>
+  <visual>
+    <origin xyz="0.100032 -0.242316 -0.032068" rpy="0 0 0"/>
+    <geometry>
+      <mesh filename="package://rover_description/meshes/basketback_v1_1.stl" scale="0.001 0.001 0.001"/>
+    </geometry>
+    <material name="silver"/>
+  </visual>
+  <!-- <collision>
+    <origin xyz="0.100032 -0.242316 -0.032068" rpy="0 0 0"/>
+    <geometry>
+      <mesh filename="package://rover_description/meshes/basketback_v1_1.stl" scale="0.001 0.001 0.001"/>
+    </geometry>
+  </collision> -->
+</link>
+<link name="Part23_v1_1">
+  <inertial>
+    <origin xyz="0.131396858909605 0.01402351974986385 -0.21656709357141518" rpy="0 0 0"/>
+    <mass value="0.042580149813532274"/>
+    <inertia ixx="0.001" iyy="0.001" izz="0.001" ixy="0.0" iyz="0.0" ixz="-0.0"/>
+  </inertial>
+  <visual>
+    <origin xyz="0.259143 -0.22803 -0.247532" rpy="0 0 0"/>
+    <geometry>
+      <mesh filename="package://rover_description/meshes/Part23_v1_1.stl" scale="0.001 0.001 0.001"/>
+    </geometry>
+    <material name="silver"/>
+  </visual>
+  <!-- <collision>
+    <origin xyz="0.259143 -0.22803 -0.247532" rpy="0 0 0"/>
+    <geometry>
+      <mesh filename="package://rover_description/meshes/Part23_v1_1.stl" scale="0.001 0.001 0.001"/>
+    </geometry>
+  </collision> -->
+</link>
+<link name="wahaczv2_v1_1">
+  <inertial>
+    <origin xyz="-0.023176555814518024 -4.1320900287522555e-07 -0.04511955865856667" rpy="0 0 0"/>
+    <mass value="0.07043737243020472"/>
+    <inertia ixx="0.001" iyy="0.001" izz="0.001" ixy="-0.0" iyz="-0.0" ixz="-8e-06"/>
+  </inertial>
+  <visual>
+    <origin xyz="0.141705 -0.242206 -0.012202" rpy="0 0 0"/>
+    <geometry>
+      <mesh filename="package://rover_description/meshes/wahaczv2_v1_1.stl" scale="0.001 0.001 0.001"/>
+    </geometry>
+    <material name="silver"/>
+  </visual>
+  <!-- <collision>
+    <origin xyz="0.141705 -0.242206 -0.012202" rpy="0 0 0"/>
+    <geometry>
+      <mesh filename="package://rover_description/meshes/wahaczv2_v1_1.stl" scale="0.001 0.001 0.001"/>
+    </geometry>
+  </collision> -->
+</link>
+<link name="Part23_v1__1__1">
+  <inertial>
+    <origin xyz="0.017838722629285486 -0.00015248025011649347 -0.01105791490528938" rpy="0 0 0"/>
+    <mass value="0.042580149813532274"/>
+    <inertia ixx="0.001" iyy="0.001" izz="0.001" ixy="-0.0" iyz="0.0" ixz="0.0"/>
+  </inertial>
+  <visual>
+    <origin xyz="0.160676 -0.242206 0.042537" rpy="0 0 0"/>
+    <geometry>
+      <mesh filename="package://rover_description/meshes/Part23_v1__1__1.stl" scale="0.001 0.001 0.001"/>
+    </geometry>
+    <material name="silver"/>
+  </visual>
+  <!-- <collision>
+    <origin xyz="0.160676 -0.242206 0.042537" rpy="0 0 0"/>
+    <geometry>
+      <mesh filename="package://rover_description/meshes/Part23_v1__1__1.stl" scale="0.001 0.001 0.001"/>
+    </geometry>
+  </collision> -->
+</link>
+<link name="felga_v1_1">
+  <inertial>
+    <origin xyz="-0.012459222389996541 -4.1432309669242606e-07 0.0001754141402649373" rpy="0 0 0"/>
+    <mass value="0.1074921153953226"/>
+    <inertia ixx="0.001" iyy="0.001" izz="0.001" ixy="-0.0" iyz="0.0" ixz="0.001"/>
+  </inertial>
+  <visual>
+    <origin xyz="0.124074 -0.242206 0.067554" rpy="0 0 0"/>
+    <geometry>
+      <mesh filename="package://rover_description/meshes/felga_v1_1.stl" scale="0.001 0.001 0.001"/>
+    </geometry>
+    <material name="silver"/>
+  </visual>
+  <!-- <collision>
+    <origin xyz="0.124074 -0.242206 0.067554" rpy="0 0 0"/>
+    <geometry>
+      <mesh filename="package://rover_description/meshes/felga_v1_1.stl" scale="0.001 0.001 0.001"/>
+    </geometry>
+  </collision> -->
+</link>
+<link name="basketback_v1__1__1">
+  <inertial>
+    <origin xyz="0.026034774004740982 0.006999585676523312 -0.014715061794331689" rpy="0 0 0"/>
+    <mass value="0.05211230478294979"/>
+    <inertia ixx="0.001" iyy="0.001" izz="0.001" ixy="0.0" iyz="-0.0" ixz="-0.0"/>
+  </inertial>
+  <visual>
+    <origin xyz="-0.100093 -0.235316 -0.039506" rpy="0 0 0"/>
+    <geometry>
+      <mesh filename="package://rover_description/meshes/basketback_v1__1__1.stl" scale="0.001 0.001 0.001"/>
+    </geometry>
+    <material name="silver"/>
+  </visual>
+  <!-- <collision>
+    <origin xyz="-0.100093 -0.235316 -0.039506" rpy="0 0 0"/>
+    <geometry>
+      <mesh filename="package://rover_description/meshes/basketback_v1__1__1.stl" scale="0.001 0.001 0.001"/>
+    </geometry>
+  </collision> -->
+</link>
+<link name="Part23_v1__2__1">
+  <inertial>
+    <origin xyz="0.1283716107326754 -0.008031348396453863 -0.23724592322337062" rpy="0 0 0"/>
+    <mass value="0.042580149813532274"/>
+    <inertia ixx="0.001" iyy="0.001" izz="0.001" ixy="0.0" iyz="-0.0" ixz="0.0"/>
+  </inertial>
+  <visual>
+    <origin xyz="0.000782 -0.250609 -0.262371" rpy="0 0 0"/>
+    <geometry>
+      <mesh filename="package://rover_description/meshes/Part23_v1__2__1.stl" scale="0.001 0.001 0.001"/>
+    </geometry>
+    <material name="silver"/>
+  </visual>
+  <!-- <collision>
+    <origin xyz="0.000782 -0.250609 -0.262371" rpy="0 0 0"/>
+    <geometry>
+      <mesh filename="package://rover_description/meshes/Part23_v1__2__1.stl" scale="0.001 0.001 0.001"/>
+    </geometry>
+  </collision> -->
+</link>
+<link name="wahaczv2_v1__1__1">
+  <inertial>
+    <origin xyz="0.021899536448331536 -4.1543758552697874e-07 -0.04575306339461184" rpy="0 0 0"/>
+    <mass value="0.07043737243020472"/>
+    <inertia ixx="0.001" iyy="0.001" izz="0.001" ixy="-0.0" iyz="0.0" ixz="0.001"/>
+  </inertial>
+  <visual>
+    <origin xyz="-0.141015 -0.242426 -0.005977" rpy="0 0 0"/>
+    <geometry>
+      <mesh filename="package://rover_description/meshes/wahaczv2_v1__1__1.stl" scale="0.001 0.001 0.001"/>
+    </geometry>
+    <material name="silver"/>
+  </visual>
+  <!-- <collision>
+    <origin xyz="-0.141015 -0.242426 -0.005977" rpy="0 0 0"/>
+    <geometry>
+      <box size="0.03 0.029 0.095"/>
+    </geometry>
+  </collision> -->
+</link>
+<link name="Part23_v1__3__1">
+  <inertial>
+    <origin xyz="-0.01650871074358476 -0.010098348396470613 -0.018826101919743238" rpy="0 0 0"/>
+    <mass value="0.042580149813532274"/>
+    <inertia ixx="0.001" iyy="0.001" izz="0.001" ixy="-0.0" iyz="-0.0" ixz="-0.0"/>
+  </inertial>
+  <visual>
+    <origin xyz="-0.156069 -0.252816 0.040099" rpy="0 0 0"/>
+    <geometry>
+      <mesh filename="package://rover_description/meshes/Part23_v1__3__1.stl" scale="0.001 0.001 0.001"/>
+    </geometry>
+    <material name="silver"/>
+  </visual>
+  <!-- <collision>
+    <origin xyz="-0.156069 -0.252816 0.040099" rpy="0 0 0"/>
+    <geometry>
+      <mesh filename="package://rover_description/meshes/Part23_v1__3__1.stl" scale="0.001 0.001 0.001"/>
+    </geometry>
+  </collision> -->
+</link>
+<link name="felga_v1__1__1">
+  <inertial>
+    <origin xyz="0.012459250006080766 -4.143234904607773e-07 -0.00017511100317847694" rpy="0 0 0"/>
+    <mass value="0.1074921153953226"/>
+    <inertia ixx="0.001" iyy="0.001" izz="0.001" ixy="-0.0" iyz="0.0" ixz="0.001"/>
+  </inertial>
+  <visual>
+    <origin xyz="-0.120412 -0.242566 0.072351" rpy="0 0 0"/>
+    <geometry>
+      <mesh filename="package://rover_description/meshes/felga_v1__1__1.stl" scale="0.001 0.001 0.001"/>
+    </geometry>
+    <material name="silver"/>
+  </visual>
+  <!-- <collision>
+    <origin xyz="-0.120412 -0.242566 0.072351" rpy="0 0 0"/>
+    <geometry>
+      <mesh filename="package://rover_description/meshes/felga_v1__1__1.stl" scale="0.001 0.001 0.001"/>
+    </geometry>
+  </collision> -->
+</link>
+<link name="basketlewy_v1_1">
+  <inertial>
+    <origin xyz="0.006583911389326097 0.019139032837798216 -0.014290024911945354" rpy="0 0 0"/>
+    <mass value="0.05235016883934813"/>
+    <inertia ixx="0.001" iyy="0.001" izz="0.001" ixy="0.0" iyz="-0.0" ixz="-0.0"/>
+  </inertial>
+  <visual>
+    <origin xyz="-0.12 -0.025272 -0.040912" rpy="0 0 0"/>
+    <geometry>
+      <mesh filename="package://rover_description/meshes/basketlewy_v1_1.stl" scale="0.001 0.001 0.001"/>
+    </geometry>
+    <material name="silver"/>
+  </visual>
+  <!-- <collision>
+    <origin xyz="-0.12 -0.025272 -0.040912" rpy="0 0 0"/>
+    <geometry>
+      <mesh filename="package://rover_description/meshes/basketlewy_v1_1.stl" scale="0.001 0.001 0.001"/>
+    </geometry>
+  </collision> -->
+</link>
+<link name="basketlewy_v1__1__1">
+  <inertial>
+    <origin xyz="-0.006583911389325181 -0.019139861484379406 -0.014290024911945896" rpy="0 0 0"/>
+    <mass value="0.05235016883934813"/>
+    <inertia ixx="0.001" iyy="0.001" izz="0.001" ixy="0.0" iyz="0.0" ixz="0.0"/>
+  </inertial>
+  <visual>
+    <origin xyz="0.12 0.134772 -0.040912" rpy="0 0 0"/>
+    <geometry>
+      <mesh filename="package://rover_description/meshes/basketlewy_v1__1__1.stl" scale="0.001 0.001 0.001"/>
+    </geometry>
+    <material name="silver"/>
+  </visual>
+  <!-- <collision>
+    <origin xyz="0.12 0.134772 -0.040912" rpy="0 0 0"/>
+    <geometry>
+      <mesh filename="package://rover_description/meshes/basketlewy_v1__1__1.stl" scale="0.001 0.001 0.001"/>
+    </geometry>
+  </collision> -->
+</link>
+<link name="basket_v1_1">
+  <inertial>
+    <origin xyz="-0.0225178401248569 0.019120872680852132 -0.014281400761913844" rpy="0 0 0"/>
+    <mass value="0.05241217155974444"/>
+    <inertia ixx="0.001" iyy="0.001" izz="0.001" ixy="-0.0" iyz="-0.0" ixz="0.0"/>
+  </inertial>
+  <visual>
+    <origin xyz="0.106 -0.025272 -0.040912" rpy="0 0 0"/>
+    <geometry>
+      <mesh filename="package://rover_description/meshes/basket_v1_1.stl" scale="0.001 0.001 0.001"/>
+    </geometry>
+    <material name="silver"/>
+  </visual>
+  <!-- <collision>
+    <origin xyz="0.106 -0.025272 -0.040912" rpy="0 0 0"/>
+    <geometry>
+      <mesh filename="package://rover_description/meshes/basket_v1_1.stl" scale="0.001 0.001 0.001"/>
+    </geometry>
+  </collision> -->
+</link>
+<link name="basket_v1__1__1">
+  <inertial>
+    <origin xyz="0.0225178401248549 -0.019121701327435486 -0.014281400761914486" rpy="0 0 0"/>
+    <mass value="0.05241217155974444"/>
+    <inertia ixx="0.001" iyy="0.001" izz="0.001" ixy="-0.0" iyz="0.0" ixz="-0.0"/>
+  </inertial>
+  <visual>
+    <origin xyz="-0.106 0.134772 -0.040912" rpy="0 0 0"/>
+    <geometry>
+      <mesh filename="package://rover_description/meshes/basket_v1__1__1.stl" scale="0.001 0.001 0.001"/>
+    </geometry>
+    <material name="silver"/>
+  </visual>
+  <!-- <collision>
+    <origin xyz="-0.106 0.134772 -0.040912" rpy="0 0 0"/>
+    <geometry>
+      <mesh filename="package://rover_description/meshes/basket_v1__1__1.stl" scale="0.001 0.001 0.001"/>
+    </geometry>
+  </collision> -->
+</link>
+<link name="Part23_v1__4__1">
+  <inertial>
+    <origin xyz="0.13253630698400776 -0.0099003483962612 -0.03737455851107026" rpy="0 0 0"/>
+    <mass value="0.042580149813532274"/>
+    <inertia ixx="0.001" iyy="0.001" izz="0.001" ixy="0.0" iyz="-0.0" ixz="0.0"/>
+  </inertial>
+  <visual>
+    <origin xyz="0.00434 -0.054434 -0.064294" rpy="0 0 0"/>
+    <geometry>
+      <mesh filename="package://rover_description/meshes/Part23_v1__4__1.stl" scale="0.001 0.001 0.001"/>
+    </geometry>
+    <material name="silver"/>
+  </visual>
+  <!-- <collision>
+    <origin xyz="0.00434 -0.054434 -0.064294" rpy="0 0 0"/>
+    <geometry>
+      <mesh filename="package://rover_description/meshes/Part23_v1__4__1.stl" scale="0.001 0.001 0.001"/>
+    </geometry>
+  </collision> -->
+</link>
+<link name="Part23_v1__5__1">
+  <inertial>
+    <origin xyz="0.13448630698400552 -0.009900348396264053 0.16066944148892914" rpy="0 0 0"/>
+    <mass value="0.042580149813532274"/>
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
File: install/rover_description/share/rover_description/urdf/materials.xacro (robot description, xacro)
@@ -1 +1,6 @@
-/home/pawla/ros2_ws/src/rover_description/rover_description/urdf/materials.xacro
+<?xml version="1.0" ?>
+<robot name="Rover" xmlns:xacro="http://www.ros.org/wiki/xacro" >
+<material name="silver">
+  <color rgba="0.700 0.700 0.700 1.000"/>
+</material>
+</robot>
