Commit message: zmiana kinematyki

File: src/rover_description/rover_description/urdf/Rover.xacro (robot description, xacro)
@@ -1051,5 +1051,5 @@
   <axis xyz="-0.014057 0.0 -0.999901"/>
   <dynamics damping="0.1" friction="0.1"/>
-  <limit effort="100" lower="-0.785398" upper="0.785398" velocity="10"/>
+  <limit effort="100" lower="-1.5708" upper="1.5708" velocity="10"/>
 </joint>
 <joint name="Rigid 16" type="fixed">
@@ -1083,5 +1083,5 @@
   <axis xyz="-0.014057 0.0 -0.999901"/>
   <dynamics damping="0.1" friction="0.1"/>
-  <limit effort="100" lower="-0.785398" upper="0.785398" velocity="10"/>
+  <limit effort="100" lower="-1.5708" upper="1.5708" velocity="10"/>
 </joint>
 <joint name="Rigid 21" type="fixed">
@@ -1145,5 +1145,5 @@
   <axis xyz="-0.0 0.0 -1.0"/>
   <dynamics damping="0.1" friction="0.1"/>
-  <limit effort="100" lower="-0.785398" upper="0.785398" velocity="10"/>
+  <limit effort="100" lower="-1.5708" upper="1.5708" velocity="10"/>
 </joint>
 <!-- TYL LEWY -->
@@ -1154,5 +1154,5 @@
   <axis xyz="0.0 0.0 -1.0"/>
   <dynamics damping="0.1" friction="0.1"/>
-  <limit effort="100" lower="-0.785398" upper="0.785398" velocity="10"/>
+  <limit effort="100" lower="-1.5708" upper="1.5708" velocity="10"/>
 </joint>
 <!-- SRODEK PRAWY -->
@@ -1163,5 +1163,5 @@
   <axis xyz="0.0 0.0 -1.0"/>
   <dynamics damping="0.1" friction="0.1"/>
-  <limit effort="100" lower="-0.785398" upper="0.785398" velocity="10"/>
+  <limit effort="100" lower="-1.5708" upper="1.5708" velocity="10"/>
 </joint>
 <!-- TYL PRAWY -->
@@ -1172,5 +1172,5 @@
   <axis xyz="-0.0 0.0 -1.0"/>
   <dynamics damping="0.1" friction="0.1"/>
-  <limit effort="100" lower="-0.785398" upper="0.785398" velocity="10"/>
+  <limit effort="100" lower="-1.5708" upper="1.5708" velocity="10"/>
 </joint>
 <joint name="Rigid 35" type="fixed">
